Commit message: ros1 version of rb1 simulation

File: my_rb1_description/urdf/my_rb1_robot.urdf (robot description, URDF)
Before this commit: robot rb1_robot, 7 links, 6 joints
Links:
- link back_caster: mass None -> 0.5
- link base_link: mass None -> 20.5; geometry collision cylinder length=0.3 radius=0.25; visual cylinder length=0.3 radius=0.25
- link front_caster: mass None -> 0.5
- link front_laser: geometry 
- link left_wheel: mass None -> 1.5; geometry collision cylinder length=0.03 radius=0.025; visual cylinder length=0.03 radius=0.025
- link right_wheel: mass None -> 1.5; geometry collision cylinder length=0.03 radius=0.025; visual cylinder length=0.03 radius=0.025
Joints:
- joint base_link_back_caster_joint: origin xyz=0.1 0 -0.15 rpy=0 0 0 -> xyz=-0.1 0.0 -0.15 rpy=0 0 0
- joint base_link_front_caster_joint: origin xyz=-0.1 0 -0.15 rpy=0 0 0 -> xyz=0.1 0.0 -0.15 rpy=0 0 0
- joint base_link_front_laser_joint: origin xyz=0.25 0 0.08 rpy=0 0 0 -> xyz=0.25 0 0.075 rpy=3.14 0 0
- joint base_link_left_wheel_joint: limit effort=10000 velocity=1000 -> (none); origin xyz=0 0.2 -.15 rpy=0 0 0 -> xyz=0 0.2 -0.15 rpy=0 0 0
- joint base_link_plate_joint: origin xyz=0 0 .175 rpy=0 0 0 -> xyz=0 0 0.15 rpy=0 0 0
- joint base_link_right_wheel_joint: limit effort=10000 velocity=1000 -> (none); origin xyz=0 -0.2 -.15 rpy=0 0 0 -> xyz=0 -0.2 -0.15 rpy=0 0 0
